File: Tremolo.sch (KiCad schematic (older format))
At the start: 110 parts, among them J1 Input, J10 R1, J11 R2, J12 TRG, J13 GND, J1A1 LeftA, J1B1 LeftB, J1C1 LeftC, J2 GND, J2A1 SwitchA, J2B1 SwitchB, J2C1 SwitchC, J3 +9v, J3A1 RightA, J3B1 RightB, J3C1 RightC, J4 GND, J5 RateSlv, J6 Gnd, J7 L2, J8 L1, J9 RateTip, Q1 BC549C, Q2 BC549C, Q3 BC549C, Q4 J113, Q5 BC549C, Q6 BC549C, T1 LeftTr, T2 RightTr, U1 TL072, U2 TL072, U3 TL072, U4 TL074, U5 VACTL, U6 VACTR

Commit message: V2.0 provisionaly completed
Parts:
- removed J1A1: LeftA, Connector_Wire:SolderWire-0.25sqmm_1x03_P4.2mm_D0.65mm_OD1.7mm, symbol Connector_Generic:Conn_01x03
- removed J1B1: LeftB, Connector_Wire:SolderWire-0.25sqmm_1x03_P4.2mm_D0.65mm_OD1.7mm, symbol Connector_Generic:Conn_01x03
- removed J1C1: LeftC, Connector_Wire:SolderWire-0.25sqmm_1x03_P4.2mm_D0.65mm_OD1.7mm, symbol Connector_Generic:Conn_01x03
- removed J2A1: SwitchA, Connector_Wire:SolderWire-0.25sqmm_1x03_P4.2mm_D0.65mm_OD1.7mm, symbol Connector_Generic:Conn_01x03
- removed J2B1: SwitchB, Connector_Wire:SolderWire-0.25sqmm_1x03_P4.2mm_D0.65mm_OD1.7mm, symbol Connector_Generic:Conn_01x03
- removed J2C1: SwitchC, Connector_Wire:SolderWire-0.25sqmm_1x03_P4.2mm_D0.65mm_OD1.7mm, symbol Connector_Generic:Conn_01x03
- removed J3A1: RightA, Connector_Wire:SolderWire-0.25sqmm_1x03_P4.2mm_D0.65mm_OD1.7mm, symbol Connector_Generic:Conn_01x03
- removed J3B1: RightB, Connector_Wire:SolderWire-0.25sqmm_1x03_P4.2mm_D0.65mm_OD1.7mm, symbol Connector_Generic:Conn_01x03
- removed J3C1: RightC, Connector_Wire:SolderWire-0.25sqmm_1x03_P4.2mm_D0.65mm_OD1.7mm, symbol Connector_Generic:Conn_01x03
- removed U5: VACTL, OptoDevice:PerkinElmer_VTL5C, symbol Isolator:VTL5C
- removed U6: VACTR, OptoDevice:PerkinElmer_VTL5C, symbol Isolator:VTL5C
- added J14: LSB1, Connector_Wire:SolderWire-0.25sqmm_1x01_D0.65mm_OD1.7mm, symbol Connector_Generic:Conn_01x01
- added J15: RSA1, Connector_Wire:SolderWire-0.25sqmm_1x01_D0.65mm_OD1.7mm, symbol Connector_Generic:Conn_01x01
- added J16: LSB2, Connector_Wire:SolderWire-0.25sqmm_1x01_D0.65mm_OD1.7mm, symbol Connector_Generic:Conn_01x01
- added J17: RSA2, Connector_Wire:SolderWire-0.25sqmm_1x01_D0.65mm_OD1.7mm, symbol Connector_Generic:Conn_01x01
- added J18: RSA3, Connector_Wire:SolderWire-0.25sqmm_1x01_D0.65mm_OD1.7mm, symbol Connector_Generic:Conn_01x01
- added J19: LSB3, Connector_Wire:SolderWire-0.25sqmm_1x01_D0.65mm_OD1.7mm, symbol Connector_Generic:Conn_01x01
- added J20: LSA1, Connector_Wire:SolderWire-0.25sqmm_1x01_D0.65mm_OD1.7mm, symbol Connector_Generic:Conn_01x01
- added J21: RSB1, Connector_Wire:SolderWire-0.25sqmm_1x01_D0.65mm_OD1.7mm, symbol Connector_Generic:Conn_01x01
- added J22: LSA3, Connector_Wire:SolderWire-0.25sqmm_1x01_D0.65mm_OD1.7mm, symbol Connector_Generic:Conn_01x01
- added J23: RSB3, Connector_Wire:SolderWire-0.25sqmm_1x01_D0.65mm_OD1.7mm, symbol Connector_Generic:Conn_01x01
- added J24: LSA2, Connector_Wire:SolderWire-0.25sqmm_1x01_D0.65mm_OD1.7mm, symbol Connector_Generic:Conn_01x01
- added J25: RSB2, Connector_Wire:SolderWire-0.25sqmm_1x01_D0.65mm_OD1.7mm, symbol Connector_Generic:Conn_01x01
- added J26: SWA1, Connector_Wire:SolderWire-0.25sqmm_1x01_D0.65mm_OD1.7mm, symbol Connector_Generic:Conn_01x01
- added J27: SWA2, Connector_Wire:SolderWire-0.25sqmm_1x01_D0.65mm_OD1.7mm, symbol Connector_Generic:Conn_01x01
- added J28: SWA3, Connector_Wire:SolderWire-0.25sqmm_1x01_D0.65mm_OD1.7mm, symbol Connector_Generic:Conn_01x01
- added J29: SWB1, Connector_Wire:SolderWire-0.25sqmm_1x01_D0.65mm_OD1.7mm, symbol Connector_Generic:Conn_01x01
- added J30: SWB2, Connector_Wire:SolderWire-0.25sqmm_1x01_D0.65mm_OD1.7mm, symbol Connector_Generic:Conn_01x01
- added J31: SWB3, Connector_Wire:SolderWire-0.25sqmm_1x01_D0.65mm_OD1.7mm, symbol Connector_Generic:Conn_01x01
- added VLD1, VRD1: D_Photo, MyLibrary:LED_D5.0mm, symbol MyGlobalLibrary:D_Photo
- added VLR1, VRR1: D_LDR, MyLibrary:R_LDR_5.2x5.2mm_P3.5mm_Horizontal, symbol MyGlobalLibrary:D_LDR
- Q1, Q2, Q3, Q4, Q5, Q6: footprint Package_TO_SOT_THT:TO-92L_Inline_Wide -> MyLibrary:TO-92L_Inline_Wide
- renumbered D3 to DL3, D2 to DR2
Connections:
- net GND: now also J18.1 (Pin_1), J19.1 (Pin_1); no longer U1.5 (+), U3.5 (+)
- net MODE11: now also J21.1 (Pin_1)
- net Shape12: now also RV4.1; no longer RV4.3
- net Shape4: now also RV3.1; no longer RV3.3
- net VDC: now also U1.5 (+), U3.5 (+)
- net at Q1.3 (E), R8.1: now also C5.2, R9.1
- net at C7.2, C8.2, R8.2: no longer C5.2, R9.1
- net at C7.1, R17.1: now also J20.1 (Pin_1)
- net at R17.2, R23.1: now also J24.1 (Pin_1)
- net at R18.2, R24.1: now also J25.1 (Pin_1)
- net at C14.1, R25.2, R29.1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: now also RV1.1; no longer RV1.3
- net at C15.1, R27.2, R30.1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: now also RV2.1; no longer RV2.3
- net at T2.3 (SA): now also J30.1 (Pin_1)
- net at T2.4 (SB): now also J27.1 (Pin_1)
- net at J10.1 (Pin_1): now also J26.1 (Pin_1), J31.1 (Pin_1)
- net at J11.1 (Pin_1): now also J28.1 (Pin_1), J29.1 (Pin_1)
- net at R5.2: now also J17.1 (Pin_1)
- net at R4.2: now also J16.1 (Pin_1)
- net at R32.2: now also RV3.3; no longer RV3.1
- net at R35.2: now also RV4.3; no longer RV4.1
- net LA1: no longer names the net of D5.1 (K)
- net LA1: now also VLD1.2 (A)
- net LA2: no longer names the net of DL3.1 (K), Q2.1 (C)
- net LA2: now also VLD1.1 (K)
- net LB1: no longer names the net of C14.2, R23.2, R25.1, U2.2 (-)
- net LB1: now also VLR1.2
- net LB2: no longer names the net of RV1.2
- net LB2: now also RV1.3, VLR1.1; no longer RV1.1
- net RA1: no longer names the net of D4.1 (K)
- net RA1: now also VRD1.2 (A)
- net RA2: no longer names the net of DR2.1 (K), Q3.1 (C)
- net RA2: now also VRD1.1 (K)
- net RB1: no longer names the net of C15.2, R24.2, R27.1, U2.6 (-)
- net RB1: now also VRR1.1
- net RB2: no longer names the net of RV2.2
- net RB2: now also RV2.3, VRR1.2; no longer RV2.1
- no-connect marks 13 -> 4
Other:
- note removed: "PADS"
- note removed: "VACTROLS"
- moved on the sheet: C5, R10, R9
